File: hardware/USB_Saturn_obdev.sch (KiCad schematic (older format))
At the start: 19 parts, among them CON1 AVR-ISP-6, J1 USB_B, J2 CONN_01X09, J3 CONN_01X09, U1 ATMEGA328-PU, X1 12M

Commit message: Added backup library
Changed logos
Parts:
- CON1: footprint Pin_Headers:Pin_Header_Straight_2x03_Pitch2.00mm -> Pin_Headers:Pin_Header_Straight_2x03_Pitch2.54mm
Changed lines of the file:
@@
 F 0 "CON1" H 6445 2890 50  0000 C CNN
 F 1 "AVR-ISP-6" H 6285 2420 50  0000 L BNN
-F 2 "Pin_Headers:Pin_Header_Straight_2x03_Pitch2.00mm" V 6030 2690 50  0001 C CNN
+F 2 "Pin_Headers:Pin_Header_Straight_2x03_Pitch2.54mm" V 6030 2690 50  0001 C CNN
 F 3 "" H 6525 2650 50  0001 C CNN
 	1    6550 2650

Commit message: Kicad format changes
Parts:
- C1, C5: footprint Capacitors_THT:CP_Radial_D4.0mm_P2.00mm -> Capacitor_THT:CP_Radial_D4.0mm_P2.00mm; symbol device:CP1 -> USB_Saturn_obdev-rescue:CP1-device
- C2: footprint Capacitors_THT:C_Disc_D3.0mm_W1.6mm_P2.50mm -> Capacitor_THT:C_Disc_D3.4mm_W2.1mm_P2.50mm; symbol device:C -> USB_Saturn_obdev-rescue:C-device
- C3, C4: footprint Capacitors_THT:C_Disc_D3.4mm_W2.1mm_P2.50mm -> Capacitor_THT:C_Disc_D3.4mm_W2.1mm_P2.50mm; symbol device:C_Small -> USB_Saturn_obdev-rescue:C_Small-device
- CON1: footprint Pin_Headers:Pin_Header_Straight_2x03_Pitch2.54mm -> Connector_PinHeader_2.54mm:PinHeader_2x03_P2.54mm_Vertical; symbol atmel:AVR-ISP-6 -> USB_Saturn_obdev-rescue:AVR-ISP-6-atmel
- D1, D2: footprint Diodes_THT:D_T-1_P5.08mm_Horizontal -> Diode_THT:D_T-1_P5.08mm_Horizontal; symbol device:D_Zener -> USB_Saturn_obdev-rescue:D_Zener-device
- J1: footprint Connectors:USB_B -> Connector_USB:USB_B_OST_USB-B1HSxx_Horizontal; symbol conn:USB_B -> USB_Saturn_obdev-rescue:USB_B-conn
- R1, R2, R3, R4: footprint Resistors_THT:R_Axial_DIN0207_L6.3mm_D2.5mm_P10.16mm_Horizontal -> Resistor_THT:R_Axial_DIN0207_L6.3mm_D2.5mm_P10.16mm_Horizontal; symbol device:R -> USB_Saturn_obdev-rescue:R-device
- R5, R6: footprint Resistors_THT:R_Axial_DIN0207_L6.3mm_D2.5mm_P10.16mm_Horizontal -> Resistor_THT:R_Axial_DIN0207_L6.3mm_D2.5mm_P10.16mm_Horizontal; symbol device:R_Small -> USB_Saturn_obdev-rescue:R_Small-device
- U1: footprint Housings_DIP:DIP-28_W7.62mm -> Package_DIP:DIP-28_W7.62mm; symbol atmel:ATMEGA328-PU -> USB_Saturn_obdev-rescue:ATMEGA328-PU-atmel
- X1: footprint Crystals:Crystal_HC49-4H_Vertical -> Crystal:Crystal_HC49-4H_Vertical; symbol device:Crystal -> USB_Saturn_obdev-rescue:Crystal-device
Changed lines of the file:
@@
 EESchema Schematic File Version 4
 LIBS:USB_Saturn_obdev-cache
-EELAYER 26 0
+EELAYER 29 0
 EELAYER END
 $Descr A4 11693 8268
@@
 $EndDescr
 $Comp
-L atmel:ATMEGA328-PU U1
+L USB_Saturn_obdev-rescue:ATMEGA328-PU-atmel U1
 U 1 1 599F8C9A
 P 2800 3800
 F 0 "U1" H 2050 5050 50  0000 L BNN
 F 1 "ATMEGA328-PU" H 3200 2400 50  0000 L BNN
-F 2 "Housings_DIP:DIP-28_W7.62mm" H 2800 3800 50  0001 C CIN
+F 2 "Package_DIP:DIP-28_W7.62mm" H 2800 3800 50  0001 C CIN
 F 3 "" H 2800 3800 50  0001 C CNN
 	1    2800 3800
@@
 $EndComp
 $Comp
-L conn:USB_B J1
+L USB_Saturn_obdev-rescue:USB_B-conn J1
 U 1 1 599F903E
 P 7600 4550
 F 0 "J1" H 7400 5000 50  0000 L CNN
 F 1 "USB_B" H 7400 4900 50  0000 L CNN
-F 2 "Connectors:USB_B" H 7750 4500 50  0001 C CNN
+F 2 "Connector_USB:USB_B_OST_USB-B1HSxx_Horizontal" H 7750 4500 50  0001 C CNN
 F 3 "" H 7750 4500 50  0001 C CNN
 	1    7600 4550
@@
 $EndComp
 $Comp
-L device:R R2
+L USB_Saturn_obdev-rescue:R-device R2
 U 1 1 599F9150
 P 5550 4500
 F 0 "R2" V 5630 4500 50  0000 C CNN
 F 1 "48o" V 5550 4500 50  0000 C CNN
-F 2 "Resistors_THT:R_Axial_DIN0207_L6.3mm_D2.5mm_P10.16mm_Horizontal" V 5480 4500 50  0001 C CNN
+F 2 "Resistor_THT:R_Axial_DIN0207_L6.3mm_D2.5mm_P10.16mm_Horizontal" V 5480 4500 50  0001 C CNN
 F 3 "" H 5550 4500 50  0001 C CNN
 	1    5550 4500
@@
 $EndComp
 $Comp
-L device:R R3
+L USB_Saturn_obdev-rescue:R-device R3
 U 1 1 599F9200
 P 5550 4700
 F 0 "R3" V 5630 4700 50  0000 C CNN
 F 1 "48o" V 5550 4700 50  0000 C CNN
-F 2 "Resistors_THT:R_Axial_DIN0207_L6.3mm_D2.5mm_P10.16mm_Horizontal" V 5480 4700 50  0001 C CNN
+F 2 "Resistor_THT:R_Axial_DIN0207_L6.3mm_D2.5mm_P10.16mm_Horizontal" V 5480 4700 50  0001 C CNN
 F 3 "" H 5550 4700 50  0001 C CNN
 	1    5550 4700
@@
 $EndComp
 $Comp
-L device:R R4
+L USB_Saturn_obdev-rescue:R-device R4
 U 1 1 599F945D
 P 6300 4350
 F 0 "R4" V 6200 4350 50  0000 C CNN
 F 1 "1k5" V 6300 4350 50  0000 C CNN
-F 2 "Resistors_THT:R_Axial_DIN0207_L6.3mm_D2.5mm_P10.16mm_Horizontal" V 6230 4350 50  0001 C CNN
+F 2 "Resistor_THT:R_Axial_DIN0207_L6.3mm_D2.5mm_P10.16mm_Horizontal" V 6230 4350 50  0001 C CNN
 F 3 "" H 6300 4350 50  0001 C CNN
 	1    6300 4350
@@
 NoConn ~ 1900 3300
 $Comp
-L device:C C2
+L USB_Saturn_obdev-rescue:C-device C2
 U 1 1 599FA76C
 P 1700 3150
 F 0 "C2" H 1725 3250 50  0000 L CNN
 F 1 "0u1" H 1725 3050 50  0000 L CNN
-F 2 "Capacitors_THT:C_Disc_D3.0mm_W1.6mm_P2.50mm" H 1738 3000 50  0001 C CNN
+F 2 "Capacitor_THT:C_Disc_D3.4mm_W2.1mm_P2.50mm" H 1738 3000 50  0001 C CNN
 F 3 "" H 1700 3150 50  0001 C CNN
 	1    1700 3150
@@
 $EndComp
 $Comp
-L device:CP1 C1
+L USB_Saturn_obdev-rescue:CP1-device C1
 U 1 1 599FA7B3
 P 1200 3150
 F 0 "C1" H 1000 3250 50  0000 L CNN
 F 1 "10u" H 1000 3050 50  0000 L CNN
-F 2 "Capacitors_THT:CP_Radial_D4.0mm_P2.00mm" H 1200 3150 50  0001 C CNN
+F 2 "Capacitor_THT:CP_Radial_D4.0mm_P2.00mm" H 1200 3150 50  0001 C CNN
 F 3 "" H 1200 3150 50  0001 C CNN
 	1    1200 3150
@@
 NoConn ~ 1900 3000
 $Comp
-L device:R R1
+L USB_Saturn_obdev-rescue:R-device R1
 U 1 1 599FC04B
 P 4700 4150
 F 0 "R1" V 4780 4150 50  0000 C CNN
 F 1 "22k" V 4700 4150 50  0000 C CNN
-F 2 "Resistors_THT:R_Axial_DIN0207_L6.3mm_D2.5mm_P10.16mm_Horizontal" V 4630 4150 50  0001 C CNN
+F 2 "Resistor_THT:R_Axial_DIN0207_L6.3mm_D2.5mm_P10.16mm_Horizontal" V 4630 4150 50  0001 C CNN
 F 3 "" H 4700 4150 50  0001 C CNN
 	1    4700 4150
@@
 NoConn ~ 3800 5000
 $Comp
-L device:Crystal X1
+L USB_Saturn_obdev-rescue:Crystal-device X1
 U 1 1 599FD1AA
 P 4800 3350
 F 0 "X1" H 4800 3200 50  0000 C CNN
 F 1 "12M" V 4800 3350 50  0000 C CNN
-F 2 "Crystals:Crystal_HC49-4H_Vertical" H 4800 3350 50  0001 C CNN
+F 2 "Crystal:Crystal_HC49-4H_Vertical" H 4800 3350 50  0001 C CNN
 F 3 "" H 4800 3350 50  0001 C CNN
 	1    4800 3350
@@
 $EndComp
 $Comp
-L device:C_Small C3
+L USB_Saturn_obdev-rescue:C_Small-device C3
 U 1 1 599FD268
 P 5100 3200
 F 0 "C3" H 5110 3270 50  0000 L CNN
 F 1 "10n" V 5000 3150 50  0000 L CNN
-F 2 "Capacitors_THT:C_Disc_D3.4mm_W2.1mm_P2.50mm" H 5100 3200 50  0001 C CNN
+F 2 "Capacitor_THT:C_Disc_D3.4mm_W2.1mm_P2.50mm" H 5100 3200 50  0001 C CNN
 F 3 "" H 5100 3200 50  0001 C CNN
 	1    5100 3200
@@
 $EndComp
 $Comp
-L device:C_Small C4
+L USB_Saturn_obdev-rescue:C_Small-device C4
 U 1 1 599FD363
 P 5100 3500
 F 0 "C4" H 5110 3570 50  0000 L CNN
 F 1 "10n" V 5000 3450 50  0000 L CNN
-F 2 "Capacitors_THT:C_Disc_D3.4mm_W2.1mm_P2.50mm" H 5100 3500 50  0001 C CNN
+F 2 "Capacitor_THT:C_Disc_D3.4mm_W2.1mm_P2.50mm" H 5100 3500 50  0001 C CNN
 F 3 "" H 5100 3500 50  0001 C CNN
 	1    5100 3500
@@
 SCK
 $Comp
-L device:D_Zener D1
+L USB_Saturn_obdev-rescue:D_Zener-device D1
 U 1 1 599FD921
 P 6000 4900
 F 0 "D1" H 6000 5000 50  0000 C CNN
 F 1 "3v6" H 6000 4800 50  0000 C CNN
-F 2 "Diodes_THT:D_T-1_P5.08mm_Horizontal" H 6000 4900 50  0001 C CNN
+F 2 "Diode_THT:D_T-1_P5.08mm_Horizontal" H 6000 4900 50  0001 C CNN
 F 3 "" H 6000 4900 50  0001 C CNN
 	1    6000 4900
@@
 $EndComp
 $Comp
-L device:D_Zener D2
+L USB_Saturn_obdev-rescue:D_Zener-device D2
 U 1 1 599FD9C5
 P 6300 4900
 F 0 "D2" H 6300 5000 50  0000 C CNN
 F 1 "3v6" H 6300 4800 50  0000 C CNN
-F 2 "Diodes_THT:D_T-1_P5.08mm_Horizontal" H 6300 4900 50  0001 C CNN
+F 2 "Diode_THT:D_T-1_P5.08mm_Horizontal" H 6300 4900 50  0001 C CNN
 F 3 "" H 6300 4900 50  0001 C CNN
 	1    6300 4900
@@
 	6000 2200 6000 2100
 $Comp
-L atmel:AVR-ISP-6 CON1
+L USB_Saturn_obdev-rescue:AVR-ISP-6-atmel CON1
 U 1 1 59A0074F
 P 6550 2650
 F 0 "CON1" H 6445 2890 50  0000 C CNN
 F 1 "AVR-ISP-6" H 6285 2420 50  0000 L BNN
-F 2 "Pin_Headers:Pin_Header_Straight_2x03_Pitch2.54mm" V 6030 2690 50  0001 C CNN
+F 2 "Connector_PinHeader_2.54mm:PinHeader_2x03_P2.54mm_Vertical" V 6030 2690 50  0001 C CNN
 F 3 "" H 6525 2650 50  0001 C CNN
 	1    6550 2650
@@
 	4250 4150 4350 4050
 $Comp
-L device:R_Small R5
+L USB_Saturn_obdev-rescue:R_Small-device R5
 U 1 1 59A07354
 P 9000 3800
 F 0 "R5" H 8875 3825 50  0000 L CNN
 F 1 "22k" H 8825 3750 50  0000 L CNN
-F 2 "Resistors_THT:R_Axial_DIN0207_L6.3mm_D2.5mm_P10.16mm_Horizontal" H 9000 3800 50  0001 C CNN
+F 2 "Resistor_THT:R_Axial_DIN0207_L6.3mm_D2.5mm_P10.16mm_Horizontal" H 9000 3800 50  0001 C CNN
 F 3 "" H 9000 3800 50  0001 C CNN
 	1    9000 3800
@@
 $EndComp
 $Comp
-L device:R_Small R6
+L USB_Saturn_obdev-rescue:R_Small-device R6
 U 1 1 59A07412
 P 9300 3800
 F 0 "R6" H 9325 3825 50  0000 L CNN
 F 1 "22k" H 9325 3750 50  0000 L CNN
-F 2 "Resistors_THT:R_Axial_DIN0207_L6.3mm_D2.5mm_P10.16mm_Horizontal" H 9300 3800 50  0001 C CNN
+F 2 "Resistor_THT:R_Axial_DIN0207_L6.3mm_D2.5mm_P10.16mm_Horizontal" H 9300 3800 50  0001 C CNN
 F 3 "" H 9300 3800 50  0001 C CNN
 	1    9300 3800
@@
 D-
 $Comp
-L device:CP1 C5
+L USB_Saturn_obdev-rescue:CP1-device C5
 U 1 1 59AC2F83
 P 1450 3150
 F 0 "C5" H 1250 3250 50  0000 L CNN
 F 1 "10u" H 1250 3050 50  0000 L CNN
-F 2 "Capacitors_THT:CP_Radial_D4.0mm_P2.00mm" H 1450 3150 50  0001 C CNN
+F 2 "Capacitor_THT:CP_Radial_D4.0mm_P2.00mm" H 1450 3150 50  0001 C CNN
 F 3 "" H 1450 3150 50  0001 C CNN
 	1    1450 3150
